File: NodeMcu/NodeMcu.kicad_pcb (KiCad board)
At the start: 2 copper layers, 8.2 x 5 mm, 38 parts, among them J1 Conn_01x15_Male, J2 Conn_01x15_Male, P1 USB_C_Plug_USB2.0, Q1 Q_Dual_NPN_NPN_E1B1C2E2B2C1, SW1 SW_Push, SW2 SW_Push, U1 ESP-12E, U2 SPX3819M5-L-3-3, U3 CH340C

Commit message: nodemcu
Parts:
- removed P1: USB_C_Plug_USB2.0, Connector_USB:USB_C_Plug_JAE_DX07P024AJ1
- added J3: USB_C_Receptacle_USB2.0, Connector_USB:USB_C_Receptacle_HRO_TYPE-C-31-M-12, F.Cu at (141.3, 67.7)
- added Q2: Q_NPN_BEC, Package_TO_SOT_SMD:SOT-23, F.Cu at (130.1, 59.6)
- J1, J2: footprint Connector_DIN:DIN41612_B_1x32_Male_Horizontal_THT -> Connector_PinHeader_2.54mm:PinHeader_1x15_P2.54mm_Vertical
- Q1: value Q_Dual_NPN_NPN_E1B1C2E2B2C1 -> Q_NPN_BEC
- SW1, SW2: footprint Button_Switch_THT:SW_PUSH_6mm -> Button_Switch_SMD:SW_SPST_FSMSM
- moved U1 73.1 mm to (104.1, 64.0), turned to 90 degrees
- moved SW2 63.3 mm to (137.9, 59.6)
- moved J1 63.0 mm to (129.7, 76.6), turned to -90 degrees
- moved J2 59.5 mm to (129.7, 52.0), turned to -90 degrees
- moved SW1 57.2 mm to (137.9, 75.6)
- moved U3 55.3 mm to (123.8, 60.1)
- moved R17 45.2 mm to (102.7, 73.8), turned to 180 degrees
- moved R16 44.8 mm to (96.2, 73.8), turned to 180 degrees
- moved R6 36.1 mm to (104.8, 73.8)
- moved C8 30.5 mm to (100.7, 73.8), turned to 180 degrees
- moved C1 29.2 mm to (122.3, 71.0)
- moved R10 27.0 mm to (120.8, 73.8), turned to 180 degrees
- moved R11 26.1 mm to (113.2, 54.3)
- moved D4 21.9 mm to (129.9, 71.3), turned to -90 degrees
- moved R8 20.7 mm to (123.2, 73.8)
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Connections:
- C1 pad 2: +3V3 -> GND
- C2 pad 2: +3V3 -> GND
- C3 pad 2: +3V3 -> GND
- C4 pad 1: +3V3 -> GND
- C5 pad 2: +3V3 -> GND
- C6 pad 2: +3V3 -> GND
- C7 pad 2: +3V3 -> GND
- C8 pad 1: +3V3 -> GND
- Q1 pad 3: /GPIO0 -> /nRST
- R11 pad 2: +3V3 -> GND
- R14 pad 1: Net-(Q1-Pad2) -> Net-(Q1-Pad1)
- R15 pad 2: Net-(Q1-Pad1) -> Net-(Q1-Pad2)
- R17 pad 2: +3V3 -> GND
- SW1 pad 2: +3V3 -> GND
- SW2 pad 2: +3V3 -> GND
- U1 pad 15: +3V3 -> GND
- U2 pad 2: +3V3 -> GND
- U3 pad 1: +3V3 -> GND
- U3 pad 14: Net-(Q1-Pad1) -> Net-(Q1-Pad2)
Routing:
- net +3V3: track 0.00 -> 100.1 mm, vias 0 -> 2
- net /GPIO16: track 0.00 -> 70.6 mm, vias 0 -> 4
- net /nRST: track 0.00 -> 50.2 mm, vias 0 -> 3
- net /TXD: track 0.00 -> 43.4 mm, vias 0 -> 1
- net /GPIO0: track 0.00 -> 36.7 mm, vias 0 -> 5
- net /RXD: track 0.00 -> 36.6 mm, vias 0 -> 1
- net +5VD: track 0.00 -> 26.4 mm
- net /EN: track 0.00 -> 25.7 mm
- net GND: track 0.00 -> 24.0 mm
- net /GPIO13: track 0.00 -> 21.5 mm, vias 0 -> 1
- net Net-(J3-PadA7): track 0.00 -> 21.4 mm, vias 0 -> 2
- net Net-(J3-PadA6): track 0.00 -> 21.3 mm, vias 0 -> 2
- net /GPIO12: track 0.00 -> 21.2 mm, vias 0 -> 1
- net /GPIO14: track 0.00 -> 21.1 mm, vias 0 -> 1
- net /VDDUSB: track 0.00 -> 19.1 mm
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Other:
- board size 8.2 x 5 mm -> 53 x 29 mm

Commit message: add cu
Parts:
- moved R6 1.36 mm to (106.2, 73.8)
- moved R17 0.97 mm to (103.7, 73.8)
- moved J3 0.61 mm to (140.7, 67.6)
Routing:
- net /EN: track 25.7 -> 23.0 mm
- net /ADC: track 12.3 -> 13.7 mm
- net +3V3: track 100.1 -> 98.7 mm
- net GND: track 24.0 -> 25.1 mm, vias 0 -> 22
- net Net-(J3-PadA6): track 21.3 -> 20.7 mm
- net Net-(J3-PadA7): track 21.4 -> 20.8 mm
- net /VDDUSB: track 19.1 -> 18.5 mm
- net /GPIO0: track 36.7 -> 36.2 mm, vias 5 -> 4
- added copper zone on B.Cu, net GND
- added copper zone on F.Cu, net GND

Commit message: bom gerber
Parts:
- added C9: 10uf, Capacitor_SMD:C_0402_1005Metric, F.Cu at (119.0, 60.7)
- C1: value C_Polarized -> 100uf
- C2, C7: value C -> 10uf
- C3, C4: value C -> 100nf
- C5: value C -> 1uf
- C6, C8: value C -> 470pf
- D1: value LED -> 3.3
- D2: value LED -> TXD
- D3: value LED -> RXD
- D4: footprint Diode_SMD:D_SMA -> Diode_SMD:D_SMF
- J1: value Conn_01x15_Male -> J1
- J2: value Conn_01x15_Male -> J2
- J3: value USB_C_Receptacle_USB2.0 -> usbc
- Q1: value Q_NPN_BEC -> q1
- Q2: value Q_NPN_BEC -> q2
- R1, R12, R13, R7, R9: value R -> 470
- R10, R11, R14, R15, R2, R3: value R -> 12K
- R16: value R -> 220K(1%)
- R17: value R -> 100K(1%)
- R4, R5: value R -> 1k
- R6: value R -> 12k
- R8: value R -> 0
- moved D4 0.22 mm to (129.7, 71.2)
- moved C4 0.08 mm to (119.0, 59.5), turned to 180 degrees
Connections:
- C2 pad 1: +5VD -> +3V3
- C3 pad 1: +5VD -> +3V3
- C4 pad 1: GND -> +3V3
- C4 pad 2: Net-(C4-Pad2) -> GND
- U3 pad 16: +5VD -> +3V3
- U3 pad 4: Net-(C4-Pad2) -> +3V3
Routing:
- net +5VD: track 26.4 -> 11.0 mm
- net +3V3: track 98.7 -> 111.6 mm, vias 2 -> 3
- net Net-(C4-Pad2): track 1.98 -> 0.00 mm
- net /VDDUSB: track 18.5 -> 19.1 mm
Other:
- board text added: "3.3"
- board text added: "5v"
- board text added: "ADC"
- board text added: "ADC EX"
- board text added: "D0"
- board text added: "D1"
- board text added: "D10"
- board text added: "D2"
- board text added: "D3"
- board text added: "D4"
- board text added: "D5"
- board text added: "D6"
- board text added: "D7"
- board text added: "D8"
- board text added: "D9"
- board text added: "EN"
- board text added: "ESP-12 NodeMcu Design by stone"
- board text added: "GND"
- board text added: "J1"
- board text added: "Keep on going never give up. It is never too late to learn Every man is his own worst enemy"
- board text added: "nRST"

Commit message: finish
Parts:
- C1: footprint Capacitor_Tantalum_SMD:CP_EIA-7132-28_AVX-C_Pad2.72x3.50mm_HandSolder -> lc_lib:CASE-B_3528
- D4: footprint Diode_SMD:D_SMF -> Diode_SMD:D_SOD-123
- Q1, Q2: footprint Package_TO_SOT_SMD:SOT-23 -> Package_TO_SOT_SMD:TSOT-23
- R16: value 220K(1%) -> 220K
- R17: value 100K(1%) -> 100K
- SW1, SW2: footprint Button_Switch_SMD:SW_SPST_FSMSM -> myFootPrint:SMD,3x4x2mm
- U3: footprint Package_SO:SOIC-16_3.9x9.9mm_P1.27mm -> lc_lib:SOP-16_150MIL
- moved J3 3.20 mm to (137.5, 67.4)
- moved SW1 1.54 mm to (136.5, 75.0)
- moved SW2 1.40 mm to (136.5, 59.8)
- moved Q1 0.53 mm to (130.0, 66.2)
- moved D4 0.33 mm to (129.7, 71.5)
- moved R15 0.32 mm to (129.0, 62.8)
- moved R14 0.32 mm to (131.0, 62.8)
- moved U3 0.28 mm to (123.6, 60.1), turned to -90 degrees
- moved C1 0.26 mm to (122.5, 70.9), turned to 180 degrees
- moved Q2 0.06 mm to (130.0, 59.6)
Routing:
- net +3V3: track 111.6 -> 114.3 mm
- net /VDDUSB: track 19.1 -> 16.7 mm
- net GND: track 25.1 -> 27.4 mm, vias 22 -> 14
- net Net-(R7-Pad2): track 13.6 -> 15.4 mm
- net /nRST: track 50.2 -> 51.5 mm
- net Net-(R9-Pad2): track 5.42 -> 5.96 mm
Other:
- board size 53 x 29 mm -> 49 x 29 mm
