File: NodeMcu/NodeMcu.kicad_pcb (KiCad board)
At the start: 2 copper layers, 49 x 29 mm, 40 parts, among them J1 J1, J2 J2, J3 usbc, Q1 q1, Q2 q2, SW1 SW_Push, SW2 SW_Push, U1 ESP-12E, U2 SPX3819M5-L-3-3, U3 CH340C

Commit message: update screen
Routing:
- net +3V3: track 114.3 -> 108.2 mm
Changed lines of the file:
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@@
   (segment (start 119.48 59.5) (end 119.48 60.7) (width 0.25) (layer "F.Cu") (net 1))
   (segment (start 118.275 61.905) (end 119.48 60.7) (width 0.25) (layer "F.Cu") (net 1))
-  (segment (start 115.634511 75.425489) (end 114.435 76.625) (width 0.4) (layer "F.Cu") (net 1))
   (segment (start 128.475489 50.750489) (end 108.014511 50.750489) (width 0.4) (layer "F.Cu") (net 1))
   (segment (start 108.014511 50.750489) (end 106.815 51.95) (width 0.4) (layer "F.Cu") (net 1))
@@
   (segment (start 128.815 55.6505) (end 128.815 54.3995) (width 0.4) (layer "F.Cu") (net 1))
   (segment (start 119.4 68.075) (end 119.4 67.2) (width 0.4) (layer "F.Cu") (net 1))
-  (segment (start 119.515 76.625) (end 118.315489 75.425489) (width 0.4) (layer "F.Cu") (net 1))
   (segment (start 106.71 54.3) (end 107.6 54.3) (width 0.4) (layer "F.Cu") (net 1))
   (segment (start 121 70.9) (end 121 73.14) (width 0.4) (layer "F.Cu") (net 1))
@@
   (segment (start 129.675 51.95) (end 128.475489 50.750489) (width 0.4) (layer "F.Cu") (net 1))
   (segment (start 128.8095 54.405) (end 128.815 54.3995) (width 0.4) (layer "F.Cu") (net 1))
-  (segment (start 118.315489 75.425489) (end 115.634511 75.425489) (width 0.4) (layer "F.Cu") (net 1))
   (segment (start 121 73.14) (end 120.29 73.85) (width 0.4) (layer "F.Cu") (net 1))
   (segment (start 128.7455 55.68) (end 128.775 55.6505) (width 0.25) (layer "F.Cu") (net 1))
