File: NodeMcu/NodeMcu.kicad_sch (KiCad schematic)
At the start: 38 parts, among them J1 Conn_01x15_Male, J2 Conn_01x15_Male, P1 USB_C_Plug_USB2.0, Q1 Q_Dual_NPN_NPN_E1B1C2E2B2C1, SW1 SW_Push, SW2 SW_Push, U1 ESP-12E, U2 SPX3819M5-L-3-3, U3 CH340C

Commit message: nodemcu
Parts:
- removed P1: USB_C_Plug_USB2.0, Connector_USB:USB_C_Plug_JAE_DX07P024AJ1, symbol Connector:USB_C_Plug_USB2.0
- removed Q1: Q_Dual_NPN_NPN_E1B1C2E2B2C1, Package_TO_SOT_SMD:SOT-23, symbol Device:Q_Dual_NPN_NPN_E1B1C2E2B2C1
- added J3: USB_C_Receptacle_USB2.0, Connector_USB:USB_C_Receptacle_HRO_TYPE-C-31-M-12, symbol Connector:USB_C_Receptacle_USB2.0
- added Q1, Q2: Q_NPN_BEC, Package_TO_SOT_SMD:SOT-23, symbol Device:Q_NPN_BEC
- J1, J2: footprint Connector_DIN:DIN41612_B_1x32_Male_Horizontal_THT -> Connector_PinHeader_2.54mm:PinHeader_1x15_P2.54mm_Vertical
- SW1, SW2: footprint Button_Switch_THT:SW_PUSH_6mm -> Button_Switch_SMD:SW_SPST_FSMSM
Connections:
- net VUSB is gone; now on net VDDUSB: J1.1 (Pin_1)
- net +3V3: no longer C1.2, C2.2, C3.2, C4.1, C5.2, C6.2, C7.2, C8.1, J1.2 (Pin_2), J1.6 (Pin_6), J1.8 (Pin_8), J2.2 (Pin_2), J2.9 (Pin_9), R11.2, R17.2, SW1.2, SW2.2, U1.15 (GND), U2.2 (GND), U3.1 (GND)
- net GPIO0: now also Q2.3 (C)
- net VDDUSB: now also J3.A4 (VBUS), J3.A9 (VBUS), J3.B4 (VBUS), J3.B9 (VBUS)
- net nRST: now also Q1.3 (C)
- net at R14.2, U3.13 (~{DTR}): now also Q2.2 (E)
- net at R15.2, U3.14 (~{RTS}): now also Q1.2 (E)
- net at U3.5 (UD+): now also J3.A6 (D+), J3.B6 (D+)
- net at U3.6 (UD-): now also J3.A7 (D-), J3.B7 (D-)
- net at R15.1: now also Q2.1 (B)
- net at R14.1: now also Q1.1 (B)
- new net GND: C1.2, C2.2, C3.2, C4.1, C5.2, C6.2, C7.2, C8.1, J1.2 (Pin_2), J1.6 (Pin_6), J1.8 (Pin_8), J2.2 (Pin_2), J2.9 (Pin_9), J3.A1 (GND), J3.A12 (GND), J3.B1 (GND), J3.B12 (GND), J3.S1 (SHIELD), R11.2, R17.2, SW1.2, SW2.2, U1.15 (GND), U2.2 (GND), U3.1 (GND)
- no-connect marks 18 -> 20
Other:
- note added: "KEY-LED"
- note added: "ONNECT"
- note added: "POWER"
- note added: "SP-12"
- note added: "USB-UART"
- moved on the sheet: C1, C2, C3, C4, C5, C6, C7, C8, D2, D3, D4, J1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

Commit message: bom gerber
Parts:
- added C9: 10uf, Capacitor_SMD:C_0402_1005Metric, symbol Device:C
- C1: value C_Polarized -> 100uf
- C2, C7: value C -> 10uf
- C3, C4: value C -> 100nf
- C5: value C -> 1uf
- C6, C8: value C -> 470pf
- D1: value LED -> 3.3
- D2: value LED -> TXD
- D3: value LED -> RXD
- D4: footprint Diode_SMD:D_SMA -> Diode_SMD:D_SMF
- J1: value Conn_01x15_Male -> J1
- J2: value Conn_01x15_Male -> J2
- J3: value USB_C_Receptacle_USB2.0 -> usbc
- Q1: value Q_NPN_BEC -> q1
- Q2: value Q_NPN_BEC -> q2
- R1, R12, R13, R7, R9: value R -> 470
- R10, R11, R14, R15, R2, R3: value R -> 12K
- R16: value R -> 220K(1%)
- R17: value R -> 100K(1%)
- R4, R5: value R -> 1k
- R6: value R -> 12k
- R8: value R -> 0
Connections:
- net +3V3: now also C2.1, C3.1, C4.1, U3.16 (VCC), U3.4 (V3), C9.1
- net +5VD: no longer C2.1, C3.1, U3.16 (VCC)
- net GND: now also C4.2, C9.2; no longer C4.1

Commit message: finish
Parts:
- C1: footprint Capacitor_Tantalum_SMD:CP_EIA-7132-28_AVX-C_Pad2.72x3.50mm_HandSolder -> lc_lib:CASE-B_3528
- D4: footprint Diode_SMD:D_SMF -> Diode_SMD:D_SOD-123
- Q1, Q2: footprint Package_TO_SOT_SMD:SOT-23 -> Package_TO_SOT_SMD:TSOT-23
- SW1, SW2: footprint Button_Switch_SMD:SW_SPST_FSMSM -> myFootPrint:SMD,3x4x2mm
- U3: footprint Package_SO:SOIC-16_3.9x9.9mm_P1.27mm -> lc_lib:SOP-16_150MIL
Changed lines of the file:
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@@
       (effects (font (size 1.27 1.27)) (justify left))
     )
-    (property "Footprint" "Button_Switch_SMD:SW_SPST_FSMSM" (id 2) (at 224.79 62.23 0)
+    (property "Footprint" "myFootPrint:SMD,3x4x2mm" (id 2) (at 224.79 62.23 0)
       (effects (font (size 1.27 1.27)) hide)
     )
@@
       (effects (font (size 1.27 1.27)) (justify left))
     )
-    (property "Footprint" "Package_SO:SOIC-16_3.9x9.9mm_P1.27mm" (id 2) (at 92.71 149.86 0)
+    (property "Footprint" "lc_lib:SOP-16_150MIL" (id 2) (at 92.71 149.86 0)
       (effects (font (size 1.27 1.27)) (justify left) hide)
     )
@@
       (effects (font (size 1.27 1.27)) (justify left))
     )
-    (property "Footprint" "Diode_SMD:D_SMF" (id 2) (at 57.785 115.57 0)
+    (property "Footprint" "Diode_SMD:D_SOD-123" (id 2) (at 57.785 115.57 0)
       (effects (font (size 1.27 1.27)) hide)
     )
@@
       (effects (font (size 1.27 1.27)) (justify left))
     )
-    (property "Footprint" "Package_TO_SOT_SMD:SOT-23" (id 2) (at 146.05 133.35 0)
+    (property "Footprint" "Package_TO_SOT_SMD:TSOT-23" (id 2) (at 146.05 133.35 0)
       (effects (font (size 1.27 1.27)) hide)
     )
@@
     (property "Reference" "C1" (id 0) (at 125.73 20.32 90))
     (property "Value" "100uf" (id 1) (at 128.27 22.86 90))
-    (property "Footprint" "Capacitor_Tantalum_SMD:CP_EIA-7132-28_AVX-C_Pad2.72x3.50mm_HandSolder" (id 2) (at 124.46 23.1648 0)
+    (property "Footprint" "lc_lib:CASE-B_3528" (id 2) (at 124.46 23.1648 0)
       (effects (font (size 1.27 1.27)) hide)
     )
@@
       (effects (font (size 1.27 1.27)) (justify left))
     )
-    (property "Footprint" "Button_Switch_SMD:SW_SPST_FSMSM" (id 2) (at 194.31 62.23 0)
+    (property "Footprint" "myFootPrint:SMD,3x4x2mm" (id 2) (at 194.31 62.23 0)
       (effects (font (size 1.27 1.27)) hide)
     )
@@
       (effects (font (size 1.27 1.27)) (justify left))
     )
-    (property "Footprint" "Package_TO_SOT_SMD:SOT-23" (id 2) (at 147.32 156.21 0)
+    (property "Footprint" "Package_TO_SOT_SMD:TSOT-23" (id 2) (at 147.32 156.21 0)
       (effects (font (size 1.27 1.27)) hide)
     )
@@
     )
     (path "/a7286792-287e-40c5-8151-5ba91dee889f"
-      (reference "C1") (unit 1) (value "100uf") (footprint "Capacitor_Tantalum_SMD:CP_EIA-7132-28_AVX-C_Pad2.72x3.50mm_HandSolder")
+      (reference "C1") (unit 1) (value "100uf") (footprint "lc_lib:CASE-B_3528")
     )
     (path "/7c00ca17-1b33-42c5-9d50-ea1e066e3966"
@@
     )
     (path "/4bd99efa-40aa-4b31-9466-ee87627720f0"
-      (reference "D4") (unit 1) (value "B120-E3") (footprint "Diode_SMD:D_SMF")
+      (reference "D4") (unit 1) (value "B120-E3") (footprint "Diode_SMD:D_SOD-123")
     )
     (path "/e6053544-5ba2-43e9-b1b8-fe98b78ac554"
@@
     )
     (path "/53cc671a-d4a7-43a0-aecc-08ecfea2f543"
-      (reference "Q1") (unit 1) (value "q1") (footprint "Package_TO_SOT_SMD:SOT-23")
+      (reference "Q1") (unit 1) (value "q1") (footprint "Package_TO_SOT_SMD:TSOT-23")
     )
     (path "/f3e71929-c9a1-427a-a7d6-0bc2b52c3802"
-      (reference "Q2") (unit 1) (value "q2") (footprint "Package_TO_SOT_SMD:SOT-23")
+      (reference "Q2") (unit 1) (value "q2") (footprint "Package_TO_SOT_SMD:TSOT-23")
     )
     (path "/636f1d33-6937-48b5-a3b2-7c6eee4be461"
@@
     )
     (path "/cbd93821-096f-4094-8611-620944c67ada"
-      (reference "SW1") (unit 1) (value "SW_Push") (footprint "Button_Switch_SMD:SW_SPST_FSMSM")
+      (reference "SW1") (unit 1) (value "SW_Push") (footprint "myFootPrint:SMD,3x4x2mm")
     )
     (path "/05a6d9e6-ede4-496a-a12f-0db20fb4e557"
-      (reference "SW2") (unit 1) (value "SW_Push") (footprint "Button_Switch_SMD:SW_SPST_FSMSM")
+      (reference "SW2") (unit 1) (value "SW_Push") (footprint "myFootPrint:SMD,3x4x2mm")
     )
     (path "/00000000-0000-0000-0000-000061cc7fc4"
@@
     )
     (path "/34eb6719-7713-41ef-b8d2-9cc36d38f374"
-      (reference "U3") (unit 1) (value "CH340C") (footprint "Package_SO:SOIC-16_3.9x9.9mm_P1.27mm")
-    )
-  )
+      (reference "U3") (unit 1) (value "CH340C") (footprint "lc_lib:SOP-16_150MIL")
+    )
+  )
