File: screen/screen.kicad_sch (KiCad schematic)
At the start: 34 parts, among them J1 USB_C_Receptacle_USB2.0, J2 Conn_01x02_Female, J3 Conn_01x12_Female, J4 Conn_01x06_Female, SW1 SW_DPDT_x2, SW2 SW_Push, SW3 SW_Push, U1 TP4056_[C16581], U3 SPX3819M5-L-3-3, U4 ESP-12E

Commit message: screen finish
Parts:
- C2: renamed from C7; footprint Capacitor_SMD:C_0603_1608Metric -> Capacitor_SMD:C_0402_1005Metric
- C3: renamed from C8; footprint Capacitor_SMD:C_0603_1608Metric -> Capacitor_SMD:C_0402_1005Metric
- C4: renamed from C9; footprint Capacitor_SMD:C_0603_1608Metric -> Capacitor_SMD:C_0402_1005Metric
- C5: renamed from C10; footprint Capacitor_SMD:C_0603_1608Metric -> Capacitor_SMD:C_0402_1005Metric
- C6: renamed from C2; footprint Capacitor_SMD:C_0603_1608Metric -> Capacitor_SMD:C_0402_1005Metric
- C7: renamed from C1; footprint Capacitor_SMD:C_0603_1608Metric -> Capacitor_SMD:C_0402_1005Metric
- D1: renamed from D2; footprint LED_SMD:LED_0603_1608Metric -> LED_SMD:LED_0402_1005Metric
- D2: renamed from D1; footprint LED_SMD:LED_0603_1608Metric -> LED_SMD:LED_0402_1005Metric
- D3: footprint LED_SMD:LED_0603_1608Metric -> LED_SMD:LED_0402_1005Metric
- J3: renamed from J1; footprint Connector_USB:USB_C_Receptacle_HRO_TYPE-C-31-M-12 -> digikey-footprints:USB-C_Female_Vert_DX07S024WJ3R400
- R10: renamed from R2; footprint Resistor_SMD:R_0603_1608Metric -> Resistor_SMD:R_0402_1005Metric
- R11: renamed from R3; footprint Resistor_SMD:R_0603_1608Metric -> Resistor_SMD:R_0402_1005Metric
- R12: renamed from R1; footprint Resistor_SMD:R_0603_1608Metric -> Resistor_SMD:R_0402_1005Metric
- R13: renamed from R4; footprint Resistor_SMD:R_0603_1608Metric -> Resistor_SMD:R_0402_1005Metric
- R14: renamed from R5; footprint Resistor_SMD:R_0603_1608Metric -> Resistor_SMD:R_0402_1005Metric
- renumbered C6 to C1, J3 to J1, J4 to J2, J2 to J4, R9 to R1, R10 to R2, R11 to R3, R12 to R4, R13 to R5, R14 to R6, R15 to R7, R16 to R8, R17 to R9, U3 to U1, U4 to U2, U1 to U3

Commit message: screen finish
Parts:
- R11: value 1.2K -> 2K
- R4: value 12k -> 12K
Changed lines of the file:
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@@
     (in_bom yes) (on_board yes)
     (property "Reference" "R4" (id 0) (at 46.99 37.9222 90))
-    (property "Value" "12k" (id 1) (at 46.99 40.2336 90))
+    (property "Value" "12K" (id 1) (at 46.99 40.2336 90))
     (property "Footprint" "Resistor_SMD:R_0402_1005Metric" (id 2) (at 46.99 41.402 90)
       (effects (font (size 1.27 1.27)) hide)
@@
       (effects (font (size 1.27 1.27)) (justify left))
     )
-    (property "Value" "1.2K" (id 1) (at 146.05 134.62 90)
+    (property "Value" "2K" (id 1) (at 146.05 134.62 90)
       (effects (font (size 1.27 1.27)) (justify left))
     )
@@
     )
     (path "/3de96e30-a9f9-42fe-9f9f-8683dbd508fe"
-      (reference "R4") (unit 1) (value "12k") (footprint "Resistor_SMD:R_0402_1005Metric")
+      (reference "R4") (unit 1) (value "12K") (footprint "Resistor_SMD:R_0402_1005Metric")
     )
     (path "/be4f891a-2d26-46e4-9ac3-affe2f45978a"
@@
     )
     (path "/e30cd634-f4d2-4240-ba82-7c8196230c19"
-      (reference "R11") (unit 1) (value "1.2K") (footprint "Resistor_SMD:R_0402_1005Metric")
+      (reference "R11") (unit 1) (value "2K") (footprint "Resistor_SMD:R_0402_1005Metric")
     )
     (path "/4435a727-6fc6-423a-9cd8-9f4144cc2941"

Commit message: add usb-c vi
Parts:
- J3: footprint digikey-footprints:USB-C_Female_Vert_DX07S024WJ3R400 -> My-lib-footprints:USB_C_6pin
Changed lines of the file:
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@@
       (effects (font (size 1.27 1.27)) hide)
     )
-    (property "Footprint" "digikey-footprints:USB-C_Female_Vert_DX07S024WJ3R400" (id 2) (at 39.37 132.08 0)
+    (property "Footprint" "My-lib-footprints:USB_C_6pin" (id 2) (at 39.37 132.08 0)
       (effects (font (size 1.27 1.27)) hide)
     )
@@
     )
     (path "/3f5424b0-b8ee-4018-9a47-938a3cde55c6"
-      (reference "J3") (unit 1) (value "USB_C_Receptacle_USB2.0") (footprint "digikey-footprints:USB-C_Female_Vert_DX07S024WJ3R400")
+      (reference "J3") (unit 1) (value "USB_C_Receptacle_USB2.0") (footprint "My-lib-footprints:USB_C_6pin")
     )
     (path "/db3d100b-e693-4e50-9bbc-ea30bf5d8288"
