File: esp8266/esp8266.kicad_sch (KiCad schematic)
At the start: 38 parts, among them J1 power, J2 TTL, J3 Conn_01x15_Female, J4 Conn_01x15_Female, SW1 RST, SW2 Flash, U1 ESP8266EX, U2 Flash_SOP-8_150mil, Y1 26MHz

Commit message: feat: update esp8266ex
Connections:
- net nRST is gone; now on net RST: R9.1
- net MTCK: now also U2.5 (SI); no longer U2.2 (SO)
- net MTDI: now also U2.2 (SO); no longer U2.3 (WP)
- net MTDO: now also U2.1 (CS); no longer U2.6 (CLK)
- net at R13.1: now also U2.7 (HOLD); no longer U2.1 (CS)
- net at R15.1: now also U2.6 (CLK); no longer U2.7 (HOLD)
- net at R14.1: now also U2.3 (WP); no longer U2.5 (SI)
Changed lines of the file:
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@@
     (effects (font (size 1.27 1.27)) (justify right bottom))
   )
-  (label "nRST" (at 215.9 41.91 270)
+  (label "RST" (at 215.9 41.91 270)
     (effects (font (size 1.27 1.27)) (justify right bottom))
   )

Commit message: feat 1. add 2.4G wifi  2. update esp8266 board
Parts:
- E1: footprint TRACE_ANTENNA_2.4GHZ_15.2MM -> My-lib-footprints:RF_2.4GHZ_15.2MM
Changed lines of the file:
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@@
       (effects (font (size 1.143 1.143)) (justify left))
     )
-    (property "Footprint" "TRACE_ANTENNA_2.4GHZ_15.2MM" (id 2) (at 26.67 46.99 0)
+    (property "Footprint" "My-lib-footprints:RF_2.4GHZ_15.2MM" (id 2) (at 26.67 46.99 0)
       (effects (font (size 0.508 0.508)) hide)
     )
@@
     )
     (path "/26860590-79bf-4bfc-9098-a910d085304a"
-      (reference "E1") (unit 1) (value "ANTENNA-GROUNDEDTRACE-15.2MM") (footprint "TRACE_ANTENNA_2.4GHZ_15.2MM")
+      (reference "E1") (unit 1) (value "ANTENNA-GROUNDEDTRACE-15.2MM") (footprint "My-lib-footprints:RF_2.4GHZ_15.2MM")
     )
     (path "/54b81e61-47eb-47b3-a4fb-c738687e3421"

Commit message: feat: esp8266 gerber
Connections:
- net RXD0 is gone; now on net RXD: J4.12 (Pin_12), U1.25 (U0RXD)
- net TXD0 is gone; now on net TXD: J4.13 (Pin_13), U1.26 (U0TXD)
- net CHIP_PU: no longer J3.12 (Pin_12)
- net GPIO5: no longer J4.2 (Pin_2)
- no-connect marks 3 -> 5
Changed lines of the file:
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@@
   (no_connect (at 43.18 127))
   (no_connect (at 43.18 124.46))
+  (no_connect (at 100.33 124.46))
+  (no_connect (at 43.18 149.86))
   (no_connect (at 83.82 33.02))
   (wire (pts (xy 215.9 41.91) (xy 215.9 59.69))
@@
     (effects (font (size 1.27 1.27)) (justify right bottom))
   )
-  (label "TXD0" (at 100.33 152.4 180)
+  (label "TXD" (at 100.33 152.4 180)
     (effects (font (size 1.27 1.27)) (justify right bottom))
   )
@@
     (effects (font (size 1.27 1.27)) (justify right bottom))
   )
-  (label "GPIO5" (at 100.33 124.46 180)
-    (effects (font (size 1.27 1.27)) (justify right bottom))
-  )
   (label "MTMS" (at 120.65 71.12 180)
     (effects (font (size 1.27 1.27)) (justify right bottom))
@@
     (effects (font (size 1.27 1.27)) (justify right bottom))
   )
-  (label "RXD0" (at 120.65 53.34 180)
+  (label "RXD" (at 120.65 53.34 180)
     (effects (font (size 1.27 1.27)) (justify right bottom))
   )
@@
     (effects (font (size 1.27 1.27)) (justify left bottom))
   )
-  (label "TXD0" (at 120.65 55.88 180)
+  (label "TXD" (at 120.65 55.88 180)
     (effects (font (size 1.27 1.27)) (justify right bottom))
   )
@@
     (effects (font (size 1.27 1.27)) (justify left bottom))
   )
-  (label "RXD0" (at 100.33 149.86 180)
+  (label "RXD" (at 100.33 149.86 180)
     (effects (font (size 1.27 1.27)) (justify right bottom))
   )
@@
     (effects (font (size 1.27 1.27)) (justify right bottom))
   )
-  (label "CHIP_PU" (at 43.18 149.86 0)
-    (effects (font (size 1.27 1.27)) (justify left bottom))
-  )
   (label "TXD" (at 252.73 74.93 90)
