File: project/screen-0.98/screen-0.98.kicad_pcb (KiCad board)
At the start: 2 copper layers, 34 parts, among them J1 TFT_0.96_13, J2 Conn_01x06_Female, J3 USB_C_6pin, J4 Conn_01x02_Female, SW1 SW_DPDT_x2, SW2 SW_Push, SW3 SW_Push, U1 SPX3819M5-L-3-3, U2 ESP-12E, U3 TP4056_[C16581]

Commit message: update 0.98
Parts:
- added Q1: S8050, Package_TO_SOT_SMD:SOT-23, F.Cu at (131.0, 96.3)
- added R15: 1K, Resistor_SMD:R_0402_1005Metric, F.Cu at (134.9, 97.1)
- added R16: 12K, Resistor_SMD:R_0402_1005Metric, F.Cu at (134.9, 95.1)
- moved U2 105.9 mm to (150.8, 76.7), turned to 0 degrees
- moved J4 16.3 mm to (63.2, 50.7)
Connections:
- J1 pad 11: GND -> Net-(J1-Pad11)
- J1 pad 6: /nRST -> /GPIO2
- J1 pad 7: unconnected-(J1-Pad7) -> GND
