File: project/screen-v1.3/screen.kicad_pcb (KiCad board)
At the start: 4 copper layers, 41.9 x 30 mm, 37 parts, among them J1 TTL-connect-pin4, J2 USB_C_6pin, J3 Conn_01x02_Female, Q1 S8050, SW1 SW_DPDT_x2, SW2 SW_Push, SW3 SW_Push, U1 SPX3819M5-L-3-3, U2 ESP-12E, U3 TFT_1.3_12, U4 TP4056_[C16581]

Commit message: fix: update screen  usb-ttl
Parts:
- J1: footprint Connector_PinHeader_1.27mm:PinHeader_1x04_P1.27mm_Vertical -> Connector_PinHeader_2.00mm:PinHeader_1x05_P2.00mm_Vertical
- R14: value 100k -> 330K
- moved D2 21.4 mm to (126.9, 44.0), turned to 180 degrees
- moved D3 21.2 mm to (129.0, 44.0), turned to 180 degrees
- moved J1 3.71 mm to (137.6, 45.0)
- moved J3 3.14 mm to (135.6, 60.1), turned to 0 degrees
- moved C7 0.89 mm to (130.6, 43.5)
- moved R10 0.77 mm to (126.9, 42.9), turned to 0 degrees
- moved R12 0.70 mm to (129.0, 42.9), turned to 0 degrees
- moved J2 0.40 mm to (135.4, 51.8)
Connections:
- U4 pad 0: (no net) -> GND
Routing:
- net /EN: track 2.82 -> 57.4 mm
- net Net-(D3-Pad2): track 25.6 -> 1.04 mm, vias 2 -> 0
- net Net-(D3-Pad1): track 25.9 -> 1.61 mm, vias 2 -> 0
- net Net-(D2-Pad1): track 26.0 -> 1.78 mm, vias 2 -> 0
- net Net-(D2-Pad2): track 25.0 -> 1.04 mm, vias 2 -> 0
- net GND: track 47.8 -> 32.6 mm, vias 14 -> 15
- net +BATT: track 54.3 -> 45.3 mm
- net +3V3: track 22.0 -> 14.6 mm, vias 7 -> 8
- net /GPIO0: track 47.4 -> 44.2 mm, vias 3 -> 2
- net /nRST: track 6.72 -> 4.88 mm, vias 1 -> 0
- net Net-(C6-Pad2): track 30.5 -> 32.1 mm
- net /RXD: track 33.3 -> 34.7 mm
- net Net-(R7-Pad2): track 9.63 -> 8.26 mm
- net /TXD: track 34.6 -> 35.9 mm
Other:
- board text added: "-"
- board text added: "EN"
- board text removed: "BT-"

Commit message: update
Routing:
- net +BATT: track 45.3 -> 46.4 mm
- net /EN: track 57.4 -> 56.4 mm
- net Net-(Q1-Pad3): track 22.1 -> 21.4 mm
- net /RXD: track 34.7 -> 34.1 mm
- net /TXD: track 35.9 -> 35.4 mm
